File: Schematics/Schematics.kicad_pcb (KiCad board)
At the start: 2 copper layers, 76 x 70 mm, 18 parts, among them U1 SDCardModule, U2 RecButton, U3 SetButton, U4 Display, U5 DS3231

Commit message: Updated PCB
Routing:
- net Net-(A1-Pad16): track 34.0 -> 28.3 mm
- net Net-(A1-Pad8): track 33.0 -> 28.9 mm
- net Net-(A1-Pad14): track 14.9 -> 11.4 mm
Changed lines of the file:
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@@
   (segment (start 81.075 116.325) (end 89.514511 107.885489) (width 0.25) (layer "B.Cu") (net 6))
   (segment (start 79.975 116.325) (end 81.075 116.325) (width 0.25) (layer "B.Cu") (net 6))
-  (segment (start 87.924211 85.065489) (end 87.265489 85.724211) (width 0.25) (layer "B.Cu") (net 7))
-  (segment (start 115.025 83.215) (end 114.175 82.365) (width 0.25) (layer "B.Cu") (net 7))
-  (segment (start 87.265489 85.724211) (end 87.265489 87.605489) (width 0.25) (layer "B.Cu") (net 7))
-  (segment (start 87.265489 87.605489) (end 88.39 88.73) (width 0.25) (layer "B.Cu") (net 7))
-  (segment (start 114.175 82.365) (end 96.599031 82.365) (width 0.25) (layer "B.Cu") (net 7))
-  (segment (start 96.599031 82.365) (end 93.898542 85.065489) (width 0.25) (layer "B.Cu") (net 7))
-  (segment (start 93.898542 85.065489) (end 87.924211 85.065489) (width 0.25) (layer "B.Cu") (net 7))
+  (segment (start 110.925489 87.314511) (end 89.805489 87.314511) (width 0.25) (layer "F.Cu") (net 7))
+  (segment (start 115.025 83.215) (end 110.925489 87.314511) (width 0.25) (layer "F.Cu") (net 7))
+  (segment (start 89.805489 87.314511) (end 88.39 88.73) (width 0.25) (layer "F.Cu") (net 7))
   (segment (start 88.39 91.27) (end 88.39 90.39) (width 0.25) (layer "B.Cu") (net 8))
   (segment (start 88.39 90.39) (end 75.92 77.92) (width 0.25) (layer "B.Cu") (net 8))
@@
   (segment (start 84.35 101.43) (end 75.92 93) (width 0.25) (layer "B.Cu") (net 12))
   (segment (start 88.39 101.43) (end 84.35 101.43) (width 0.25) (layer "B.Cu") (net 12))
-  (segment (start 79.975 111.245) (end 78.800489 110.070489) (width 0.25) (layer "B.Cu") (net 13))
-  (segment (start 84.829511 107.530489) (end 88.39 103.97) (width 0.25) (layer "B.Cu") (net 13))
-  (segment (start 79.488501 107.530489) (end 84.829511 107.530489) (width 0.25) (layer "B.Cu") (net 13))
-  (segment (start 78.800489 108.218501) (end 79.488501 107.530489) (width 0.25) (layer "B.Cu") (net 13))
-  (segment (start 78.800489 110.070489) (end 78.800489 108.218501) (width 0.25) (layer "B.Cu") (net 13))
+  (segment (start 79.975 111.245) (end 87.25 103.97) (width 0.25) (layer "F.Cu") (net 13))
+  (segment (start 87.25 103.97) (end 88.39 103.97) (width 0.25) (layer "F.Cu") (net 13))
   (segment (start 86.195 108.705) (end 88.39 106.51) (width 0.25) (layer "B.Cu") (net 14))
   (segment (start 79.975 108.705) (end 86.195 108.705) (width 0.25) (layer "B.Cu") (net 14))
-  (segment (start 92.14 118) (end 103.63 106.51) (width 0.25) (layer "B.Cu") (net 15))
-  (segment (start 78.800489 114.959511) (end 78.800489 117.499511) (width 0.25) (layer "B.Cu") (net 15))
-  (segment (start 78.800489 117.499511) (end 79.300978 118) (width 0.25) (layer "B.Cu") (net 15))
-  (segment (start 79.300978 118) (end 92.14 118) (width 0.25) (layer "B.Cu") (net 15))
-  (segment (start 79.975 113.785) (end 78.800489 114.959511) (width 0.25) (layer "B.Cu") (net 15))
+  (segment (start 99.215 113.785) (end 103.63 109.37) (width 0.25) (layer "F.Cu") (net 15))
+  (segment (start 79.975 113.785) (end 99.215 113.785) (width 0.25) (layer "F.Cu") (net 15))
+  (segment (start 103.63 109.37) (end 103.63 106.51) (width 0.25) (layer "F.Cu") (net 15))
   (segment (start 116.54 117) (end 116.54 109.26) (width 0.25) (layer "B.Cu") (net 19))
   (segment (start 116.54 109.26) (end 103.63 96.35) (width 0.25) (layer "B.Cu") (net 19))
